File: Reflow_Control/Reflow_Control.sch (KiCad schematic (older format))
At the start: 4 parts

Commit message: work on schematic
Parts:
- added BZ?: Buzzer, symbol Device:Buzzer
- added U?: MAX31865_Breakout, MY_FOOTPRINT:MAX31865_Breakout, symbol my_lib:MAX31865_Breakout
- U?: footprint (none) -> Package_SO:SOIC-24W_7.5x15.4mm_P1.27mm; Dist (none) -> Digikey; Dist no (none) -> 568-11907-1-ND; Man (none) -> NXP; Man no (none) -> PCA9555
Changed lines of the file:
@@
 EESchema Schematic File Version 4
+LIBS:Reflow_Control-cache
 EELAYER 26 0
 EELAYER END
@@
 L my_lib:PCA9555 U?
 U 1 1 5F6E1EB3
-P 6500 5250
-F 0 "U?" H 6500 6015 50  0000 C CNN
-F 1 "PCA9555" H 6500 5924 50  0000 C CNN
-F 2 "" H 6500 5250 50  0001 C CNN
-F 3 "" H 6500 5250 50  0001 C CNN
-	1    6500 5250
+P 3050 6750
+F 0 "U?" H 3050 7515 50  0000 C CNN
+F 1 "PCA9555" H 3050 7424 50  0000 C CNN
+F 2 "Package_SO:SOIC-24W_7.5x15.4mm_P1.27mm" H 3050 6750 50  0001 C CNN
+F 3 "" H 3050 6750 50  0001 C CNN
+F 4 "NXP" H 3050 6750 50  0001 C CNN "Man"
+F 5 "PCA9555" H 3050 6750 50  0001 C CNN "Man no"
+F 6 "Digikey" H 3050 6750 50  0001 C CNN "Dist"
+F 7 " 568-11907-1-ND " H 3050 6750 50  0001 C CNN "Dist no"
+	1    3050 6750
 	1    0    0    -1
 $EndComp
@@
 	1    0    0    -1
 $EndComp
+$Comp
+L Device:Buzzer BZ?
+U 1 1 5F6E1A0F
+P 8650 5100
+F 0 "BZ?" H 8803 5129 50  0000 L CNN
+F 1 "Buzzer" H 8803 5038 50  0000 L CNN
+F 2 "" V 8625 5200 50  0001 C CNN
+F 3 "~" V 8625 5200 50  0001 C CNN
+	1    8650 5100
+	1    0    0    -1
+$EndComp
+$Comp
+L my_lib:MAX31865_Breakout U?
+U 1 1 5F6E1D4F
+P 6050 2250
+F 0 "U?" H 6277 2346 50  0000 L CNN
+F 1 "MAX31865_Breakout" H 6277 2255 50  0000 L CNN
+F 2 "MY_FOOTPRINT:MAX31865_Breakout" H 6050 2250 50  0001 C CNN
+F 3 "" H 6050 2250 50  0001 C CNN
+	1    6050 2250
+	1    0    0    -1
+$EndComp

Commit message: work on Buzzer
Parts:
- added Q?: BC848, Package_TO_SOT_SMD:SOT-23, symbol Transistor_BJT:BC848
- added R?: 4k7, Resistor_SMD:R_1206_3216Metric_Pad1.42x1.75mm_HandSolder, symbol Device:R
- added R? (x2): 1k, Resistor_SMD:R_1206_3216Metric_Pad1.42x1.75mm_HandSolder, symbol Device:R
- BZ?: footprint (none) -> Buzzer_Beeper:Buzzer_TDK_PS1240P02BT_D12.2mm_H6.5mm; Dist (none) -> Digikey; Dist no (none) -> 445-2525-3-ND; Man (none) -> TDK; Man no (none) -> PS1240P02BT
- U?: symbol my_lib:NUCLEO-F042K6 -> Reflow_Control-rescue:NUCLEO-F042K6-my_lib
- U?: symbol my_lib:MAX31865_Breakout -> Reflow_Control-rescue:MAX31865_Breakout-my_lib
- U?: symbol my_lib:PCA9555 -> Reflow_Control-rescue:PCA9555-my_lib
- U?: symbol my_lib:SSD1306_128x64 -> Reflow_Control-rescue:SSD1306_128x64-my_lib
Connections:
- net labels added: +3.3V, Buzzer, GND
- wire segments 0 -> 11
Other:
- moved on the sheet: BZ?
Changed lines of the file:
@@
 $EndDescr
 $Comp
-L my_lib:NUCLEO-F042K6 U?
+L Reflow_Control-rescue:NUCLEO-F042K6-my_lib U?
 U 1 1 5F6E1C9D
 P 1800 6650
@@
 $EndComp
 $Comp
-L my_lib:PCA9555 U?
+L Reflow_Control-rescue:PCA9555-my_lib U?
 U 1 1 5F6E1EB3
 P 3050 6750
@@
 $EndComp
 $Comp
-L my_lib:SSD1306_128x64 U?
+L Reflow_Control-rescue:SSD1306_128x64-my_lib U?
 U 1 1 5F6E1F48
 P 9450 2850
@@
 L Device:Buzzer BZ?
 U 1 1 5F6E1A0F
-P 8650 5100
-F 0 "BZ?" H 8803 5129 50  0000 L CNN
-F 1 "Buzzer" H 8803 5038 50  0000 L CNN
-F 2 "" V 8625 5200 50  0001 C CNN
-F 3 "~" V 8625 5200 50  0001 C CNN
-	1    8650 5100
+P 8900 5300
+F 0 "BZ?" H 9053 5329 50  0000 L CNN
+F 1 "Buzzer" H 9053 5238 50  0000 L CNN
+F 2 "Buzzer_Beeper:Buzzer_TDK_PS1240P02BT_D12.2mm_H6.5mm" V 8875 5400 50  0001 C CNN
+F 3 "~" V 8875 5400 50  0001 C CNN
+F 4 "TDK" H 8900 5300 50  0001 C CNN "Man"
+F 5 "PS1240P02BT" H 8900 5300 50  0001 C CNN "Man no"
+F 6 "Digikey" H 8900 5300 50  0001 C CNN "Dist"
+F 7 "445-2525-3-ND" H 8900 5300 50  0001 C CNN "Dist no"
+	1    8900 5300
 	1    0    0    -1
 $EndComp
 $Comp
-L my_lib:MAX31865_Breakout U?
+L Reflow_Control-rescue:MAX31865_Breakout-my_lib U?
 U 1 1 5F6E1D4F
 P 6050 2250
@@
 	1    0    0    -1
 $EndComp
+$Comp
+L Transistor_BJT:BC848 Q?
+U 1 1 5F94235C
+P 8350 5700
+F 0 "Q?" H 8541 5746 50  0000 L CNN
+F 1 "BC848" H 8541 5655 50  0000 L CNN
+F 2 "Package_TO_SOT_SMD:SOT-23" H 8550 5625 50  0001 L CIN
+F 3 "http://www.infineon.com/dgdl/Infineon-BC847SERIES_BC848SERIES_BC849SERIES_BC850SERIES-DS-v01_01-en.pdf?fileId=db3a304314dca389011541d4630a1657" H 8350 5700 50  0001 L CNN
+F 4 "Nexperia" H 8350 5700 50  0001 C CNN "Man"
+F 5 "BC848B,215" H 8350 5700 50  0001 C CNN "Man no"
+F 6 "Digikey" H 8350 5700 50  0001 C CNN "Dist"
+F 7 "1727-4241-1-ND" H 8350 5700 50  0001 C CNN "Dist no"
+	1    8350 5700
+	1    0    0    -1
+$EndComp
+$Comp
+L Device:R R?
+U 1 1 5F9458E6
+P 7300 4700
+F 0 "R?" H 7370 4746 50  0000 L CNN
+F 1 "4k7" H 7370 4655 50  0000 L CNN
+F 2 "Resistor_SMD:R_1206_3216Metric_Pad1.42x1.75mm_HandSolder" V 7230 4700 50  0001 C CNN
+F 3 "~" H 7300 4700 50  0001 C CNN
+F 4 "Rhom" H 7300 4700 50  0001 C CNN "Man"
+F 5 "KTR18EZPF4701" H 7300 4700 50  0001 C CNN "Man no"
+F 6 "Digikey" H 7300 4700 50  0001 C CNN "Dist"
+F 7 "RHM4.7KAICT-ND" H 7300 4700 50  0001 C CNN "Dist no"
+	1    7300 4700
+	1    0    0    -1
+$EndComp
+$Comp
+L power:GND #PWR?
+U 1 1 5F945B67
+P 8450 6000
+F 0 "#PWR?" H 8450 5750 50  0001 C CNN
+F 1 "GND" H 8455 5827 50  0000 C CNN
+F 2 "" H 8450 6000 50  0001 C CNN
+F 3 "" H 8450 6000 50  0001 C CNN
+	1    8450 6000
+	1    0    0    -1
+$EndComp
+Wire Wire Line
+	8450 6000 8450 5900
+$Comp
+L Device:R R?
+U 1 1 5F945FB0
+P 8450 5150
+F 0 "R?" H 8520 5196 50  0000 L CNN
+F 1 "1k" H 8520 5105 50  0000 L CNN
+F 2 "Resistor_SMD:R_1206_3216Metric_Pad1.42x1.75mm_HandSolder" V 8380 5150 50  0001 C CNN
+F 3 "~" H 8450 5150 50  0001 C CNN
+F 4 "Rhom" H 8450 5150 50  0001 C CNN "Man"
+F 5 "KTR18EZPF1001" H 8450 5150 50  0001 C CNN "Man no"
+F 6 "Digikey" H 8450 5150 50  0001 C CNN "Dist"
+F 7 "RHM1.00KAICT-ND" H 8450 5150 50  0001 C CNN "Dist no"
+	1    8450 5150
+	1    0    0    -1
+$EndComp
+$Comp
+L Device:R R?
+U 1 1 5F946191
+P 7900 5700
+F 0 "R?" V 7693 5700 50  0000 C CNN
+F 1 "1k" V 7784 5700 50  0000 C CNN
+F 2 "Resistor_SMD:R_1206_3216Metric_Pad1.42x1.75mm_HandSolder" V 7830 5700 50  0001 C CNN
+F 3 "~" H 7900 5700 50  0001 C CNN
+F 4 "Rhom" H 7900 5700 50  0001 C CNN "Man"
+F 5 "KTR18EZPF1001" H 7900 5700 50  0001 C CNN "Man no"
+F 6 "Digikey" H 7900 5700 50  0001 C CNN "Dist"
+F 7 "RHM1.00KAICT-ND" H 7900 5700 50  0001 C CNN "Dist no"
+	1    7900 5700
+	0    1    1    0
+$EndComp
+Wire Wire Line
+	8450 5300 8450 5400
+Wire Wire Line
+	8450 4700 8450 4900
+Wire Wire Line
+	8800 5200 8700 5200
+Wire Wire Line
+	8700 5200 8700 4900
+Wire Wire Line
+	8700 4900 8450 4900
+Connection ~ 8450 4900
+Wire Wire Line
+	8450 4900 8450 5000
+Connection ~ 8450 5400
+Wire Wire Line
+	8450 5400 8450 5500
+Wire Wire Line
+	8450 5400 8800 5400
+$Comp
+L power:+3.3V #PWR?
+U 1 1 5F946619
+P 8450 4700
+F 0 "#PWR?" H 8450 4550 50  0001 C CNN
+F 1 "+3.3V" H 8465 4873 50  0000 C CNN
+F 2 "" H 8450 4700 50  0001 C CNN
+F 3 "" H 8450 4700 50  0001 C CNN
+	1    8450 4700
+	1    0    0    -1
+$EndComp
+Wire Wire Line
+	8050 5700 8150 5700
+Text GLabel 7650 5700 0    50   Input ~ 0
+Buzzer
+Wire Wire Line
+	7650 5700 7750 5700
 $EndSCHEMATC

Commit message: work on push buttons
Parts:
- added C? (x9): 100n, Capacitor_SMD:C_0805_2012Metric_Pad1.15x1.40mm_HandSolder, symbol Device:C
- added SW? (x7): SW_Push, Button_Switch_SMD:SW_SPST_B3S-1000, symbol Switch:SW_Push
Connections:
- net GND: now also C?.1, C?.1, C?.1, C?.1, C?.1, C?.1, C?.1, SW?.2, SW?.2, SW?.2, SW?.2, SW?.2, SW?.2, SW?.2
- net BTN_A: now reaches U?.10 (IO0_6)
- net BTN_A: now also C?.2, SW?.1
- net BTN_B: now reaches U?.11 (IO0_7)
- net BTN_B: now also C?.2, SW?.1
- net BTN_UP: now reaches U?.5 (IO0_1)
- net BTN_UP: now also C?.2, SW?.1
- net BTN_DOWN: now reaches U?.6 (IO0_2)
- net BTN_DOWN: now also C?.2, SW?.1
- net BTN_RIGHT: now reaches U?.7 (IO0_3)
- net BTN_RIGHT: now also C?.2, SW?.1
- net BTN_LEFT: now reaches U?.8 (IO0_4)
- net BTN_LEFT: now also C?.2, SW?.1
- net BTN_CENTER: now reaches U?.9 (IO0_5)
- net BTN_CENTER: now also C?.2, SW?.1
Other:
- moved on the sheet: BZ?, Q?, R?, SW?, U?

Commit message: work on rotary encoder
Parts:
- added C?: 100n, Capacitor_SMD:C_0805_2012Metric_Pad1.15x1.40mm_HandSolder, symbol Device:C
- added R?: 4k7, Resistor_SMD:R_1206_3216Metric_Pad1.42x1.75mm_HandSolder, symbol Device:R
- SW?: Dist (none) -> Digikey; Dist no (none) -> PEC11L-4220F-S0015-ND; Man (none) -> Bourns; Man no (none) -> PEC11L-4220F-S0015
Connections:
- net +3V3: now also R?.1, R?.1
- net BTN_A: now also U?.9 (IO0_5); no longer U?.10 (IO0_6)
- net BTN_B: now also U?.10 (IO0_6); no longer U?.11 (IO0_7)
- net BTN_CENTER: now also U?.8 (IO0_4); no longer U?.9 (IO0_5)
- net BTN_DOWN: now also U?.5 (IO0_1); no longer U?.6 (IO0_2)
- net BTN_LEFT: now also U?.7 (IO0_3); no longer U?.8 (IO0_4)
- net BTN_RIGHT: now also U?.6 (IO0_2); no longer U?.7 (IO0_3)
- net BTN_UP: now also U?.4 (IO0_0); no longer U?.5 (IO0_1)
- net GND: now also C?.2, C?.2, SW?.C, SW?.S2, C?.2
- net ENC_A: now reaches SW?.A
- net ENC_A: now also C?.1, R?.2, R?.2
- net ENC_B: now reaches SW?.B
- net ENC_B: now also C?.1
- net ENC_Switch: now reaches SW?.S1
- net ENC_Switch: now also U?.11 (IO0_7), C?.1
Other:
- moved on the sheet: C?, R?, SW?, U?
Changed lines of the file:
@@
 L Device:Rotary_Encoder_Switch SW?
 U 1 1 5F6E216F
-P 8150 1350
-F 0 "SW?" H 8150 1717 50  0000 C CNN
-F 1 "Rotary_Encoder_Switch" H 8150 1626 50  0000 C CNN
-F 2 "" H 8000 1510 50  0001 C CNN
-F 3 "~" H 8150 1610 50  0001 C CNN
-	1    8150 1350
+P 6800 3100
+F 0 "SW?" H 6800 3467 50  0000 C CNN
+F 1 "Rotary_Encoder_Switch" H 6800 3376 50  0000 C CNN
+F 2 "" H 6650 3260 50  0001 C CNN
+F 3 "~" H 6800 3360 50  0001 C CNN
+F 4 "Bourns" H 6800 3100 50  0001 C CNN "Man"
+F 5 "PEC11L-4220F-S0015" H 6800 3100 50  0001 C CNN "Man no"
+F 6 "Digikey" H 6800 3100 50  0001 C CNN "Dist"
+F 7 "PEC11L-4220F-S0015-ND" H 6800 3100 50  0001 C CNN "Dist no"
+	1    6800 3100
 	1    0    0    -1
 $EndComp
@@
 L Reflow_Control-rescue:MAX31865_Breakout-my_lib U?
 U 1 1 5F6E1D4F
-P 6050 2250
-F 0 "U?" H 6277 2346 50  0000 L CNN
-F 1 "MAX31865_Breakout" H 6277 2255 50  0000 L CNN
-F 2 "MY_FOOTPRINT:MAX31865_Breakout" H 6050 2250 50  0001 C CNN
-F 3 "" H 6050 2250 50  0001 C CNN
-	1    6050 2250
+P 3750 1850
+F 0 "U?" H 3977 1946 50  0000 L CNN
+F 1 "MAX31865_Breakout" H 3977 1855 50  0000 L CNN
+F 2 "MY_FOOTPRINT:MAX31865_Breakout" H 3750 1850 50  0001 C CNN
+F 3 "" H 3750 1850 50  0001 C CNN
+	1    3750 1850
 	1    0    0    -1
 $EndComp
@@
 L Device:R R?
 U 1 1 5F9458E6
-P 7450 1600
-F 0 "R?" H 7520 1646 50  0000 L CNN
-F 1 "4k7" H 7520 1555 50  0000 L CNN
-F 2 "Resistor_SMD:R_1206_3216Metric_Pad1.42x1.75mm_HandSolder" V 7380 1600 50  0001 C CNN
-F 3 "~" H 7450 1600 50  0001 C CNN
-F 4 "Rhom" H 7450 1600 50  0001 C CNN "Man"
-F 5 "KTR18EZPF4701" H 7450 1600 50  0001 C CNN "Man no"
-F 6 "Digikey" H 7450 1600 50  0001 C CNN "Dist"
-F 7 "RHM4.7KAICT-ND" H 7450 1600 50  0001 C CNN "Dist no"
-	1    7450 1600
+P 5950 2450
+F 0 "R?" H 6020 2496 50  0000 L CNN
+F 1 "4k7" H 6020 2405 50  0000 L CNN
+F 2 "Resistor_SMD:R_1206_3216Metric_Pad1.42x1.75mm_HandSolder" V 5880 2450 50  0001 C CNN
+F 3 "~" H 5950 2450 50  0001 C CNN
+F 4 "Rhom" H 5950 2450 50  0001 C CNN "Man"
+F 5 "KTR18EZPF4701" H 5950 2450 50  0001 C CNN "Man no"
+F 6 "Digikey" H 5950 2450 50  0001 C CNN "Dist"
+F 7 "RHM4.7KAICT-ND" H 5950 2450 50  0001 C CNN "Dist no"
+	1    5950 2450
 	1    0    0    -1
 $EndComp
@@
 L Device:C C?
 U 1 1 5F947CDD
-P 8400 1800
-F 0 "C?" H 8515 1846 50  0000 L CNN
-F 1 "100n" H 8515 1755 50  0000 L CNN
-F 2 "Capacitor_SMD:C_0805_2012Metric_Pad1.15x1.40mm_HandSolder" H 8438 1650 50  0001 C CNN
-F 3 "~" H 8400 1800 50  0001 C CNN
-F 4 "Samsung" H 8400 1800 50  0001 C CNN "Man"
-F 5 "CL21B104KACNNNC" H 8400 1800 50  0001 C CNN "Man nno"
-F 6 "Digikey" H 8400 1800 50  0001 C CNN "Dist"
-F 7 "1276-1099-1-ND" H 8400 1800 50  0001 C CNN "Dist no"
-	1    8400 1800
+P 6150 3400
+F 0 "C?" H 6265 3446 50  0000 L CNN
+F 1 "100n" H 6265 3355 50  0000 L CNN
+F 2 "Capacitor_SMD:C_0805_2012Metric_Pad1.15x1.40mm_HandSolder" H 6188 3250 50  0001 C CNN
+F 3 "~" H 6150 3400 50  0001 C CNN
+F 4 "Samsung" H 6150 3400 50  0001 C CNN "Man"
+F 5 "CL21B104KACNNNC" H 6150 3400 50  0001 C CNN "Man nno"
+F 6 "Digikey" H 6150 3400 50  0001 C CNN "Dist"
+F 7 "1276-1099-1-ND" H 6150 3400 50  0001 C CNN "Dist no"
+	1    6150 3400
 	1    0    0    -1
 $EndComp
@@
 L Device:C C?
 U 1 1 5F9481EB
-P 8100 2350
-F 0 "C?" H 8215 2396 50  0000 L CNN
-F 1 "100n" H 8215 2305 50  0000 L CNN
-F 2 "Capacitor_SMD:C_0805_2012Metric_Pad1.15x1.40mm_HandSolder" H 8138 2200 50  0001 C CNN
-F 3 "~" H 8100 2350 50  0001 C CNN
-F 4 "Samsung" H 8100 2350 50  0001 C CNN "Man"
-F 5 "CL21B104KACNNNC" H 8100 2350 50  0001 C CNN "Man nno"
-F 6 "Digikey" H 8100 2350 50  0001 C CNN "Dist"
-F 7 "1276-1099-1-ND" H 8100 2350 50  0001 C CNN "Dist no"
-	1    8100 2350
+P 5750 3400
+F 0 "C?" H 5865 3446 50  0000 L CNN
+F 1 "100n" H 5865 3355 50  0000 L CNN
+F 2 "Capacitor_SMD:C_0805_2012Metric_Pad1.15x1.40mm_HandSolder" H 5788 3250 50  0001 C CNN
+F 3 "~" H 5750 3400 50  0001 C CNN
+F 4 "Samsung" H 5750 3400 50  0001 C CNN "Man"
+F 5 "CL21B104KACNNNC" H 5750 3400 50  0001 C CNN "Man nno"
+F 6 "Digikey" H 5750 3400 50  0001 C CNN "Dist"
+F 7 "1276-1099-1-ND" H 5750 3400 50  0001 C CNN "Dist no"
+	1    5750 3400
 	1    0    0    -1
 $EndComp
@@
 	7350 4950 7350 5050
 Connection ~ 7350 5050
+Text GLabel 3950 6550 0    50   Output ~ 0
+BTN_UP
 Text GLabel 3950 6650 0    50   Output ~ 0
-BTN_UP
+BTN_DOWN
+Text GLabel 3950 6850 0    50   Output ~ 0
+BTN_LEFT
+Text GLabel 3950 6950 0    50   Output ~ 0
+BTN_CENTER
 Text GLabel 3950 6750 0    50   Output ~ 0
-BTN_DOWN
-Text GLabel 3950 6950 0    50   Output ~ 0
-BTN_LEFT
+BTN_RIGHT
 Text GLabel 3950 7050 0    50   Output ~ 0
-BTN_CENTER
-Text GLabel 3950 6850 0    50   Output ~ 0
-BTN_RIGHT
+BTN_A
 Text GLabel 3950 7150 0    50   Output ~ 0
-BTN_A
+BTN_B
+$Comp
+L power:GND #PWR?
+U 1 1 5F986F4B
+P 6450 3700
+F 0 "#PWR?" H 6450 3450 50  0001 C CNN
+F 1 "GND" H 6455 3527 50  0000 C CNN
+F 2 "" H 6450 3700 50  0001 C CNN
+F 3 "" H 6450 3700 50  0001 C CNN
+	1    6450 3700
+	1    0    0    -1
+$EndComp
+Wire Wire Line
+	6450 3700 6450 3650
+Wire Wire Line
+	6450 3100 6500 3100
+Wire Wire Line
+	6500 3200 6150 3200
+Wire Wire Line
+	6150 3200 6150 3250
+Wire Wire Line
+	6500 3000 6350 3000
+Wire Wire Line
+	5750 3000 5750 3250
+Wire Wire Line
+	5750 3550 5750 3650
+Wire Wire Line
+	5750 3650 6150 3650
+Connection ~ 6450 3650
+Wire Wire Line
+	6450 3650 6450 3100
+Wire Wire Line
+	6150 3550 6150 3650
+Connection ~ 6150 3650
+Wire Wire Line
+	6150 3650 6450 3650
+Text GLabel 5750 2900 1    50   Output ~ 0
+ENC_A
+Text GLabel 6150 2900 1    50   Output ~ 0
+ENC_B
+Wire Wire Line
+	5750 2900 5750 3000
+Connection ~ 5750 3000
+Wire Wire Line
+	6150 2900 6150 3200
+Connection ~ 6150 3200
+Text GLabel 7300 2900 1    50   Output ~ 0
+ENC_Switch
+$Comp
+L Device:C C?
+U 1 1 5F99A33D
+P 7300 3250
+F 0 "C?" H 7415 3296 50  0000 L CNN
+F 1 "100n" H 7415 3205 50  0000 L CNN
+F 2 "Capacitor_SMD:C_0805_2012Metric_Pad1.15x1.40mm_HandSolder" H 7338 3100 50  0001 C CNN
+F 3 "~" H 7300 3250 50  0001 C CNN
+F 4 "Samsung" H 7300 3250 50  0001 C CNN "Man"
+F 5 "CL21B104KACNNNC" H 7300 3250 50  0001 C CNN "Man nno"
+F 6 "Digikey" H 7300 3250 50  0001 C CNN "Dist"
+F 7 "1276-1099-1-ND" H 7300 3250 50  0001 C CNN "Dist no"
+	1    7300 3250
+	1    0    0    -1
+$EndComp
+$Comp
+L power:GND #PWR?
+U 1 1 5F99A3C7
+P 7300 3700
+F 0 "#PWR?" H 7300 3450 50  0001 C CNN
+F 1 "GND" H 7305 3527 50  0000 C CNN
+F 2 "" H 7300 3700 50  0001 C CNN
+F 3 "" H 7300 3700 50  0001 C CNN
+	1    7300 3700
+	1    0    0    -1
+$EndComp
+Wire Wire Line
+	7300 3700 7300 3500
+Wire Wire Line
+	7100 3200 7150 3200
+Wire Wire Line
+	7150 3200 7150 3500
+Wire Wire Line
+	7150 3500 7300 3500
+Connection ~ 7300 3500
+Wire Wire Line
+	7300 3500 7300 3400
+Wire Wire Line
+	7300 2900 7300 3000
+Wire Wire Line
+	7100 3000 7300 3000
+Connection ~ 7300 3000
+Wire Wire Line
+	7300 3000 7300 3100
 Text GLabel 3950 7250 0    50   Output ~ 0
-BTN_B
+ENC_Switch
+Wire Wire Line
+	3950 7250 4050 7250
+Wire Wire Line
+	3950 7150 4050 7150
+Wire Wire Line
+	3950 7050 4050 7050
+Wire Wire Line
+	3950 6950 4050 6950
+Wire Wire Line
+	3950 6850 4050 6850
+Wire Wire Line
+	3950 6750 4050 6750
 Wire Wire Line
 	3950 6650 4050 6650
 Wire Wire Line
-	3950 6750 4050 6750
-Wire Wire Line
-	3950 6850 4050 6850
-Wire Wire Line
-	3950 6950 4050 6950
-Wire Wire Line
-	3950 7050 4050 7050
-Wire Wire Line
-	3950 7150 4050 7150
-Wire Wire Line
-	3950 7250 4050 7250
+	3950 6550 4050 6550
+$Comp
+L Device:R R?
+U 1 1 5F9CF3CE
+P 6350 2450
+F 0 "R?" H 6420 2496 50  0000 L CNN
+F 1 "4k7" H 6420 2405 50  0000 L CNN
+F 2 "Resistor_SMD:R_1206_3216Metric_Pad1.42x1.75mm_HandSolder" V 6280 2450 50  0001 C CNN
+F 3 "~" H 6350 2450 50  0001 C CNN
+F 4 "Rhom" H 6350 2450 50  0001 C CNN "Man"
+F 5 "KTR18EZPF4701" H 6350 2450 50  0001 C CNN "Man no"
+F 6 "Digikey" H 6350 2450 50  0001 C CNN "Dist"
+F 7 "RHM4.7KAICT-ND" H 6350 2450 50  0001 C CNN "Dist no"
+	1    6350 2450
+	1    0    0    -1
+$EndComp
+Wire Wire Line
+	5950 2600 5950 3000
+Connection ~ 5950 3000
+Wire Wire Line
+	5950 3000 5750 3000
+Wire Wire Line
+	6350 2600 6350 3000
+Connection ~ 6350 3000
+Wire Wire Line
+	6350 3000 5950 3000
+$Comp
+L power:+3.3V #PWR?
+U 1 1 5F9E4634
+P 5950 2200
+F 0 "#PWR?" H 5950 2050 50  0001 C CNN
+F 1 "+3.3V" H 5965 2373 50  0000 C CNN
+F 2 "" H 5950 2200 50  0001 C CNN
+F 3 "" H 5950 2200 50  0001 C CNN
+	1    5950 2200
+	1    0    0    -1
+$EndComp
+$Comp
+L power:+3.3V #PWR?
+U 1 1 5F9E46CB
+P 6350 2200
+F 0 "#PWR?" H 6350 2050 50  0001 C CNN
+F 1 "+3.3V" H 6365 2373 50  0000 C CNN
+F 2 "" H 6350 2200 50  0001 C CNN
+F 3 "" H 6350 2200 50  0001 C CNN
+	1    6350 2200
+	1    0    0    -1
+$EndComp
+Wire Wire Line
+	6350 2200 6350 2300
+Wire Wire Line
+	5950 2300 5950 2200
 $EndSCHEMATC

Commit message: work on IO expander
Parts:
- added C?: 100n, Capacitor_SMD:C_0805_2012Metric_Pad1.15x1.40mm_HandSolder, symbol Device:C
- added JP? (x3): Jumper_3_Open, symbol Jumper:Jumper_3_Open
- added R? (x3): 4k7, Resistor_SMD:R_1206_3216Metric_Pad1.42x1.75mm_HandSolder, symbol Device:R
Connections:
- net +3V3: now also U?.24 (VCC), C?.1, JP?.1 (A), JP?.1 (A), JP?.1 (A), R?.1, R?.1, R?.1
- net GND: now also U?.12 (VSS), C?.2, JP?.3 (B), JP?.3 (B), JP?.3 (B)
- net I2C_SDA: now reaches U?.7 (D4)
- net I2C_SDA: now also U?.23 (SDA), R?.2
- net I2C_SCL: now reaches U?.8 (D5)
- net I2C_SCL: now also U?.22 (SCL), R?.2
- net INT_IO_EXP: now reaches U?.1 (INT)
- net INT_IO_EXP: now also R?.2
- net ADDR_A1: now reaches U?.2 (A1)
- net ADDR_A1: now also JP?.2 (C)
- net ADDR_A0: now reaches U?.21 (A0)
- net ADDR_A0: now also JP?.2 (C)
- net ADDR_A2: now reaches U?.3 (A2)
- net ADDR_A2: now also JP?.2 (C)
Other:
- moved on the sheet: C?, R?, SW?, U?

Commit message: work on display
Connections:
- net +3V3: now also U?.17 (3V3), U?.2 (VCC)
- net GND: now also U?.1 (GND), U?.29 (GND), U?.4 (GND)
- net I2C_SCL: now also U?.3 (SCL)
- net I2C_SDA: now also U?.4 (SDA)
Other:
- moved on the sheet: U?
Changed lines of the file:
@@
 L Reflow_Control-rescue:SSD1306_128x64-my_lib U?
 U 1 1 5F6E1F48
-P 4950 3700
-F 0 "U?" H 5427 3771 50  0000 L CNN
-F 1 "SSD1306_128x64" H 5427 3680 50  0000 L CNN
-F 2 "" H 4950 3700 50  0001 C CNN
-F 3 "" H 4950 3700 50  0001 C CNN
-	1    4950 3700
+P 8550 1000
+F 0 "U?" H 9027 1071 50  0000 L CNN
+F 1 "SSD1306_128x64" H 9027 980 50  0000 L CNN
+F 2 "" H 8550 1000 50  0001 C CNN
+F 3 "" H 8550 1000 50  0001 C CNN
+	1    8550 1000
 	1    0    0    -1
 $EndComp
@@
 	2450 3600 2000 3600
 Connection ~ 2000 3600
+$Comp
+L power:+3.3V #PWR?
+U 1 1 5FB04176
+P 3550 4150
+F 0 "#PWR?" H 3550 4000 50  0001 C CNN
+F 1 "+3.3V" H 3565 4323 50  0000 C CNN
+F 2 "" H 3550 4150 50  0001 C CNN
+F 3 "" H 3550 4150 50  0001 C CNN
+	1    3550 4150
+	1    0    0    -1
+$EndComp
+Wire Wire Line
+	3350 4200 3550 4200
+Wire Wire Line
+	3550 4200 3550 4150
+$Comp
+L power:GND #PWR?
+U 1 1 5FB0A37F
+P 2300 3250
+F 0 "#PWR?" H 2300 3000 50  0001 C CNN
+F 1 "GND" H 2305 3077 50  0000 C CNN
+F 2 "" H 2300 3250 50  0001 C CNN
+F 3 "" H 2300 3250 50  0001 C CNN
+	1    2300 3250
+	1    0    0    -1
+$EndComp
+Wire Wire Line
+	2450 3200 2300 3200
+Wire Wire Line
+	2300 3200 2300 3250
+$Comp
+L power:GND #PWR?
+U 1 1 5FB10814
+P 3550 3050
+F 0 "#PWR?" H 3550 2800 50  0001 C CNN
+F 1 "GND" H 3555 2877 50  0000 C CNN
+F 2 "" H 3550 3050 50  0001 C CNN
+F 3 "" H 3550 3050 50  0001 C CNN
+	1    3550 3050
+	1    0    0    -1
+$EndComp
+Wire Wire Line
+	3350 3000 3550 3000
+Wire Wire Line
+	3550 3000 3550 3050
+Text GLabel 7900 1050 0    50   BiDi ~ 0
+I2C_SDA
+Text GLabel 7900 1150 0    50   Input ~ 0
+I2C_SCL
+Wire Wire Line
+	7900 1050 8000 1050
+Wire Wire Line
+	7900 1150 8000 1150
+$Comp
+L power:+3.3V #PWR?
+U 1 1 5FB2BAB0
+P 7400 800
+F 0 "#PWR?" H 7400 650 50  0001 C CNN
+F 1 "+3.3V" H 7415 973 50  0000 C CNN
+F 2 "" H 7400 800 50  0001 C CNN
+F 3 "" H 7400 800 50  0001 C CNN
+	1    7400 800
+	1    0    0    -1
+$EndComp
+$Comp
+L power:GND #PWR?
+U 1 1 5FB2BB01
+P 7400 1000
+F 0 "#PWR?" H 7400 750 50  0001 C CNN
+F 1 "GND" H 7405 827 50  0000 C CNN
+F 2 "" H 7400 1000 50  0001 C CNN
+F 3 "" H 7400 1000 50  0001 C CNN
+	1    7400 1000
+	1    0    0    -1
+$EndComp
+Wire Wire Line
+	7400 1000 7400 950
+Wire Wire Line
+	7400 950  8000 950
+Wire Wire Line
+	7400 800  7400 850
+Wire Wire Line
+	7400 850  8000 850
 $EndSCHEMATC
