File: Reflow_Control/Reflow_Control.kicad_pcb (KiCad board)
At the start: 2 copper layers, 100 x 80 mm, 66 parts, among them J1 Conn_5V, J2 Conn_ssr_1, J3 Conn_ssr_2, Q1 BC848, Q2 BC848, Q3 BC848, SW1 SW_Push, SW2 SW_Push, SW3 SW_Push, SW4 SW_Push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

Commit message: work on pcb layout
Parts:
- moved U5 234.8 mm to (31.5, 33.5)
- moved SW2 223.1 mm to (256.5, 120.0)
- moved U4 222.2 mm to (106.0, 75.5), turned to 180 degrees
- moved SW3 210.8 mm to (240.0, 107.0)
- moved SW7 208.1 mm to (255.5, 107.0)
- moved U3 207.6 mm to (119.5, 100.0)
- moved SW8 207.1 mm to (239.5, 118.5)
- moved JP1 187.0 mm to (126.0, 87.5), turned to 180 degrees
- moved SW6 171.8 mm to (246.5, 89.5)
- moved R15 158.5 mm to (137.0, 72.7), turned to 270 degrees
- moved SW5 148.8 mm to (244.0, 33.0)
- moved R14 143.2 mm to (182.0, 80.5), turned to 180 degrees
- moved SW1 142.9 mm to (256.5, 72.0)
- moved R11 142.5 mm to (186.0, 74.5), turned to 180 degrees
- moved SW4 138.4 mm to (240.5, 74.0)
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Other:
- board text added: "HEATER 1"
- board text added: "HEATER 2"

Commit message: placement of display
Parts:
- moved R8 177.8 mm to (137.0, 93.5)
- moved JP3 171.0 mm to (216.5, 49.0)
- moved D2 162.5 mm to (137.5, 89.5)
- moved C11 159.0 mm to (52.7, 27.1)
- moved C2 159.0 mm to (81.0, 37.8)
- moved C3 159.0 mm to (79.3, 23.4)
- moved R1 159.0 mm to (72.0, 20.7)
- moved R2 159.0 mm to (59.9, 32.2)
- moved R3 159.0 mm to (67.8, 27.5)
- moved R5 159.0 mm to (62.3, 36.4)
- moved R7 159.0 mm to (68.7, 32.1)
- moved R9 159.0 mm to (72.7, 27.5)
- moved U1 143.8 mm to (151.2, 69.4), turned to 90 degrees
- moved JP4 142.7 mm to (146.0, 27.0)
- moved C9 134.6 mm to (250.6, 59.2)
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
Commit message: work on pcb
Parts:
- moved R3 167.7 mm to (234.5, 45.2)
- moved R7 148.0 mm to (187.0, 121.0), turned to 270 degrees
- moved R5 134.8 mm to (188.3, 84.2)
- moved C5 130.2 mm to (160.5, 117.5)
- moved H5 127.0 mm to (105.0, 92.5)
- moved C11 120.9 mm to (146.8, 103.0)
- moved H6 117.2 mm to (105.0, 117.5)
- moved R6 109.4 mm to (178.0, 85.5)
- moved R9 103.4 mm to (171.8, 57.2)
- moved C12 102.6 mm to (153.5, 117.0), turned to 180 degrees
- moved D1 94.5 mm to (187.0, 115.5), turned to 90 degrees
- moved C13 93.6 mm to (170.5, 117.5)
- moved C7 92.3 mm to (159.5, 106.2)
- moved C6 89.0 mm to (148.2, 106.5)
- moved BZ1 82.5 mm to (219.5, 38.0)
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
Commit message: Kerem & Edwin dez. 20 2020 mitarbeit
Parts:
- added C4: 100uF, Capacitor_SMD:CP_Elec_5x5.4, F.Cu at (124.2, 83.8)
- H5, H6: footprint MountingHole:MountingHole_2.5mm_Pad -> owen:MountingHole_2.5mm_Pad
- SW5: footprint Rotary_Encoder:RotaryEncoder_Alps_EC11E_Vertical_H20mm -> owen:RotaryEncoder_Alps_EC11E_Vertical_H20mm
- moved R3 123.1 mm to (121.4, 94.0)
- moved JP2 104.9 mm to (150.9, 81.3)
- moved C2 103.4 mm to (172.3, 86.3)
- moved D3 95.8 mm to (183.0, 113.0), turned to 90 degrees
- moved Q3 78.2 mm to (154.9, 56.9)
- moved R15 76.5 mm to (154.7, 53.6), turned to 180 degrees
- moved C1 73.0 mm to (159.4, 96.1)
- moved C3 68.5 mm to (119.2, 79.0), turned to 180 degrees
- moved R12 63.7 mm to (154.6, 60.7), turned to 180 degrees
- moved R9 62.3 mm to (183.0, 118.5), turned to 270 degrees
- moved BZ1 61.5 mm to (161.3, 57.9)
- moved JP1 29.6 mm to (138.7, 56.6), turned to 0 degrees
- moved U4 28.1 mm to (116.8, 83.8)
- moved H6 24.8 mm to (103.4, 92.7), turned to 90 degrees
- moved C11 24.0 mm to (170.4, 107.1)
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Connections:
- C10 pad 2: INT_ENC_B -> INT_ENC_A
- C9 pad 2: INT_ENC_A -> INT_ENC_B
- R5 pad 2: INT_ENC_A -> INT_ENC_B
- R6 pad 2: INT_ENC_B -> INT_ENC_A
- SW5 pad A: INT_ENC_A -> INT_ENC_B
- SW5 pad B: INT_ENC_B -> INT_ENC_A
- U5 pad 10: BTN_B -> BTN_RIGHT
- U5 pad 4: BTN_UP -> BTN_A
- U5 pad 5: BTN_DOWN -> BTN_LEFT
- U5 pad 6: BTN_RIGHT -> BTN_DOWN
- U5 pad 7: BTN_LEFT -> BTN_CENTER
- U5 pad 8: BTN_CENTER -> BTN_UP
- U5 pad 9: BTN_A -> BTN_B
Routing:
- net INT_ENC_B: track 0.00 -> 115.6 mm
- net INT_ENC_A: track 0.00 -> 111.9 mm
- net TIM3_CH2_HEATER_PWM: track 0.00 -> 79.3 mm
- net TIM3_CH1_HEATER_PWM: track 0.00 -> 67.3 mm
- net +3V3: track 0.00 -> 64.3 mm, vias 0 -> 23
- net I2C1_SDA: track 0.00 -> 59.5 mm
- net INT_PCA9555: track 0.00 -> 57.7 mm, vias 0 -> 2
- net SPI1_SCK: track 0.00 -> 52.3 mm, vias 0 -> 1
- net I2C1_SCL: track 0.00 -> 51.9 mm
- net Net-(D1-Pad2): track 0.00 -> 50.2 mm, vias 0 -> 2
- net BTN_A: track 0.00 -> 48.6 mm, vias 0 -> 2
- net Net-(D2-Pad2): track 0.00 -> 47.2 mm, vias 0 -> 2
- net INT_MAX31865_RDY: track 0.00 -> 46.1 mm
- net BTN_DOWN: track 0.00 -> 45.8 mm, vias 0 -> 2
- net BTN_B: track 0.00 -> 44.6 mm, vias 0 -> 2
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- added copper zone on B.Cu, net +3V3
- added copper zone on F.Cu, net +3V3

Commit message: small changes to layout
Parts:
- moved C2 21.6 mm to (154.4, 74.2)
- moved C3 0.26 mm to (119.2, 78.7)
Routing:
- net +3V3: track 64.3 -> 64.8 mm, vias 23 -> 22
Other:
- board text added: "Reflow Oven Controller"
Changed lines of the file:
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@@
-(kicad_pcb (version 20171130) (host pcbnew 5.1.5+dfsg1-2build2)
+(kicad_pcb (version 20171130) (host pcbnew 5.0.2+dfsg1-1)
   (general
     (thickness 1.6)
-    (drawings 8)
-    (tracks 362)
+    (drawings 9)
+    (tracks 361)
     (zones 0)
     (modules 67)
@@
     (47 F.CrtYd user)
     (48 B.Fab user hide)
-    (49 F.Fab user)
+    (49 F.Fab user hide)
   )
   (setup
-    (last_trace_width 0.5)
+    (last_trace_width 1)
     (user_trace_width 0.5)
     (user_trace_width 1)
@@
     (zone_45_only no)
     (trace_min 0.2)
+    (segment_width 0.2)
+    (edge_width 0.15)
     (via_size 0.8)
     (via_drill 0.4)
@@
     (uvia_min_size 0.2)
     (uvia_min_drill 0.1)
-    (edge_width 0.15)
-    (segment_width 0.2)
     (pcb_text_width 0.3)
     (pcb_text_size 1.5 1.5)
@@
   )
   (module Capacitor_SMD:C_0805_2012Metric_Pad1.15x1.40mm_HandSolder (layer F.Cu)
-    (at 172.3136 86.3092)
+    (at 154.432 74.168)
     (descr "Capacitor SMD 0805 (2012 Metric), square (rectangular) end terminal, IPC_7351 nominal with elongated pad for handsoldering. (Body size source: https://docs.google.com/spreadsheets/d/1BsfQQcO9C6DZCsRaXUlFlo91Tg2WpOkGARC1WS5S8t0/edit?usp=sharing), generated with kicad-footprint-generator")
     (tags "capacitor handsolder")
     (attr smd)
-    (fp_text reference C2 (at 0 -1.65) (layer F.SilkS)
+    (fp_text reference C2 (at 1.194 -1.61) (layer F.SilkS)
       (effects (font (size 1 1) (thickness 0.15)))
     )
@@
   )
   (module Capacitor_SMD:C_0805_2012Metric_Pad1.15x1.40mm_HandSolder (layer F.Cu)
-    (at 119.25 79 180)
+    (at 119.25 78.74 180)
     (descr "Capacitor SMD 0805 (2012 Metric), square (rectangular) end terminal, IPC_7351 nominal with elongated pad for handsoldering. (Body size source: https://docs.google.com/spreadsheets/d/1BsfQQcO9C6DZCsRaXUlFlo91Tg2WpOkGARC1WS5S8t0/edit?usp=sharing), generated with kicad-footprint-generator")
     (tags "capacitor handsolder")
@@
     (pad 1 thru_hole circle (at 0 0 90) (size 3.5 3.5) (drill 2.54) (layers *.Cu *.Mask))
   )
+  (gr_text "Reflow Oven Controller" (at 127.254 119.888) (layer F.SilkS)
+    (effects (font (size 2 2) (thickness 0.3)))
+  )
   (dimension 80 (width 0.3) (layer Dwgs.User)
     (gr_text "80.000 mm" (at 82.9 90 90) (layer Dwgs.User)
@@
   (segment (start 149.576 84.582) (end 148.209 84.582) (width 0.25) (layer F.Cu) (net 1) (status 10))
   (via (at 148.209 84.582) (size 0.8) (drill 0.4) (layers F.Cu B.Cu) (net 1))
-  (via (at 155.321 74.676) (size 0.8) (drill 0.4) (layers F.Cu B.Cu) (net 1))
-  (segment (start 155.265 74.732) (end 155.321 74.676) (width 0.25) (layer F.Cu) (net 1))
-  (segment (start 155.265 76.8) (end 155.265 74.732) (width 0.25) (layer F.Cu) (net 1) (status 10))
   (via (at 148.209 87.884) (size 0.8) (drill 0.4) (layers F.Cu B.Cu) (net 1))
   (segment (start 149.6425 87.884) (end 148.209 87.884) (width 0.25) (layer F.Cu) (net 1) (status 10))
@@
   (via (at 198.25 87.633) (size 0.8) (drill 0.4) (layers F.Cu B.Cu) (net 1))
   (via (at 122.682 67.31) (size 0.8) (drill 0.4) (layers F.Cu B.Cu) (net 1))
-  (via (at 175.0568 86.36) (size 0.8) (drill 0.4) (layers F.Cu B.Cu) (net 1))
-  (segment (start 175.006 86.3092) (end 175.0568 86.36) (width 0.25) (layer F.Cu) (net 1))
-  (segment (start 173.3386 86.3092) (end 175.006 86.3092) (width 0.25) (layer F.Cu) (net 1))
+  (via (at 156.972 74.168) (size 0.8) (drill 0.4) (layers F.Cu B.Cu) (net 1))
   (via (at 140.8 56.6) (size 0.8) (drill 0.4) (layers F.Cu B.Cu) (net 1))
   (segment (start 140.758 56.642) (end 140.8 56.6) (width 0.25) (layer F.Cu) (net 1))
@@
   (segment (start 191.8625 74.25) (end 192.0625 74.05) (width 1) (layer F.Cu) (net 1))
   (segment (start 187.75 74.25) (end 191.8625 74.25) (width 1) (layer F.Cu) (net 1))
+  (segment (start 155.265 74.24) (end 155.025 74) (width 0.25) (layer F.Cu) (net 1))
+  (segment (start 155.265 76.8) (end 155.265 74.24) (width 0.25) (layer F.Cu) (net 1))
+  (segment (start 155.193 74.168) (end 155.025 74) (width 0.25) (layer F.Cu) (net 1))
+  (segment (start 156.972 74.168) (end 155.701 74.168) (width 0.25) (layer F.Cu) (net 1))
   (segment (start 153.8745 60.706) (end 153.162 60.706) (width 0.5) (layer F.Cu) (net 2) (status 20))
   (segment (start 155.94 58.6405) (end 153.8745 60.706) (width 0.5) (layer F.Cu) (net 2))
@@
   (segment (start 168.2496 93.0496) (end 168.2496 88.8492) (width 0.25) (layer B.Cu) (net 9))
   (segment (start 192.5 104.5) (end 191.424999 103.424999) (width 0.25) (layer B.Cu) (net 9))
-  (segment (start 193.9875 92.7375) (end 192.5 91.25) (width 0.25) (layer F.Cu) (net 11))
   (segment (start 181.875 95.1) (end 181.875 92.7375) (width 0.25) (layer F.Cu) (net 10) (status 30))
   (segment (start 184.7625 92.7375) (end 187.5 90) (width 0.25) (layer F.Cu) (net 10) (status 20))
@@
   (segment (start 140.63 52.07) (end 133.739999 58.960001) (width 0.25) (layer F.Cu) (net 10))
   (segment (start 133.739999 58.960001) (end 132.94 59.76) (width 0.25) (layer F.Cu) (net 10))
+  (segment (start 193.9875 92.7375) (end 192.5 91.25) (width 0.25) (layer F.Cu) (net 11))
   (segment (start 198.25 92.7375) (end 193.9875 92.7375) (width 0.25) (layer F.Cu) (net 11) (status 10))
   (segment (start 192.5 91.25) (end 192.5 90) (width 0.25) (layer F.Cu) (net 11) (status 20))
